Commit message: update

File: ros2_ur_ws/src/pallet_gripper/urdf/pallet_gripper.urdf (robot description, URDF)
Before this commit: robot pallet_gripper, 12 links, 11 joints
Joints:
- joint J8: axis 0 1 0 -> 0.17361937 0 -0.98481283; limit lower=0 upper=0.103 effort=10 velocity=1.0 -> lower=0 upper=0.0335 effort=10 velocity=0.03; origin xyz=-0.007486 -0.0082 0.0031518 rpy=-3.14159265359 1.39629265359 -3.14159265359 -> xyz=0.014474 -0.0082 0.0031518 rpy=-3.14159265359 1.39629265359 -3.14159265359; type revolute -> prismatic
- joint J9: axis 0 1 0 -> 0.17361214 0 0.98481411; limit lower=-0.103 upper=0 effort=10 velocity=1.0 -> lower=0 upper=0.0335 effort=10 velocity=0.03; mimic joint=J8 multiplier=-1 offset=0 -> joint=J8 multiplier=1 offset=0; origin xyz=0.007486 -0.0082 0.0031518 rpy=0 1.3963 0 -> xyz=-0.014474 -0.0082 0.0031518 rpy=0 1.3963 0; type revolute -> prismatic
