Commit message: Update robot vision and hardware configuration

File: ros2_ur_ws/src/pallet/urdf/pallet.urdf (robot description, URDF)
Before this commit: robot pallet, 9 links, 8 joints
Joints:
- removed joint tool0_joint
- added joint j1: type revolute, parent base_link, child L2, origin xyz=0 0 0 rpy=1.6099 0 -1.0512, axis 0.023014 0.99974 0, limit lower=-3.14 upper=3.14 effort=5 velocity=10.471976
- joint j2: axis 0.023014 0.99974 0 -> 0 0 1; child L2 -> L3; limit lower=-3.14 upper=3.14 effort=11 velocity=10.471976 -> lower=-2.757620 upper=1.623156 effort=11 velocity=10.471976; origin xyz=0 0 0 rpy=1.6099 0 -1.0512 -> xyz=0.0012123 0.16129 0.0080631 rpy=-1.5708 0.61077 -1.5938; parent base_link -> L2
- joint j3: axis 0 0 1 -> 1 0 0; child L3 -> L4; limit lower=-2.757620 upper=1.623156 effort=5 velocity=10.471976 -> lower=-3.14 upper=0.802851 effort=5 velocity=10.471976; origin xyz=0.0012123 0.16129 0.0080631 rpy=-1.5708 0.61077 -1.5938 -> xyz=-0.2105 0 -0.0068993 rpy=1.9138 -1.5708 -0.15545; parent L2 -> L3
- joint j4: axis 1 0 0 -> 0 0 1; child L4 -> L5; limit lower=-3.14 upper=0.802851 effort=5 velocity=10.471976 -> lower=-3.14 upper=3.14 effort=1.8 velocity=10.471976; origin xyz=-0.2105 0 -0.0068993 rpy=1.9138 -1.5708 -0.15545 -> xyz=0.006 0 0.205 rpy=0 0 0.0076608; parent L3 -> L4
- joint j5: axis 0 0 1 -> 1 0 0; child L5 -> L6; limit lower=-3.14 upper=3.14 effort=1.8 velocity=10.471976 -> lower=-0.785398 upper=2.548181 effort=1.8 velocity=10.471976; origin xyz=0.006 0 0.205 rpy=0 0 0.0076608 -> xyz=0.0357 0 0.042 rpy=-0.87843 0 0; parent L4 -> L5
- joint j6: axis 1 0 0 -> 0 0 1; child L6 -> tool0; limit lower=-0.785398 upper=2.548181 effort=1.8 velocity=10.471976 -> lower=-3.14 upper=3.14 effort=1.8 velocity=10.471976; origin xyz=0.0357 0 0.042 rpy=-0.87843 0 0 -> xyz=-0.0755 0 0 rpy=0 -1.57079632679 0; parent L5 -> L6

Commit message: Align Pallet five-axis joint numbering

File: ros2_ur_ws/src/pallet/urdf/pallet.urdf (robot description, URDF)
Before this commit: robot pallet, 9 links, 8 joints
Joints:
- removed joint j6
- added joint j1: type revolute, parent base_link, child L2, origin xyz=0 0 0 rpy=1.6099 0 -1.0512, axis 0.023014 0.99974 0, limit lower=-3.14 upper=3.14 effort=11 velocity=10.471976
- joint j2: axis 0.023014 0.99974 0 -> 0 0 1; child L2 -> L3; limit lower=-3.14 upper=3.14 effort=11 velocity=10.471976 -> lower=-2.757620 upper=1.623156 effort=5 velocity=10.471976; origin xyz=0 0 0 rpy=1.6099 0 -1.0512 -> xyz=0.0012123 0.16129 0.0080631 rpy=-1.5708 0.61077 -1.5938; parent base_link -> L2
- joint j3: axis 0 0 1 -> 1 0 0; child L3 -> L4; limit lower=-2.757620 upper=1.623156 effort=5 velocity=10.471976 -> lower=-3.14 upper=0.802851 effort=1.8 velocity=10.471976; origin xyz=0.0012123 0.16129 0.0080631 rpy=-1.5708 0.61077 -1.5938 -> xyz=-0.2105 0 -0.0068993 rpy=1.9138 -1.5708 -0.15545; parent L2 -> L3
- joint j4: axis 1 0 0 -> 0 0 1; child L4 -> L5; limit lower=-3.14 upper=0.802851 effort=5 velocity=10.471976 -> lower=-3.14 upper=3.14 effort=1.8 velocity=10.471976; origin xyz=-0.2105 0 -0.0068993 rpy=1.9138 -1.5708 -0.15545 -> xyz=0.006 0 0.205 rpy=0 0 0.0076608; parent L3 -> L4
- joint j5: axis 0 0 1 -> 1 0 0; child L5 -> L6; limit lower=-3.14 upper=3.14 effort=1.8 velocity=10.471976 -> lower=-0.785398 upper=2.548181 effort=1.8 velocity=10.471976; origin xyz=0.006 0 0.205 rpy=0 0 0.0076608 -> xyz=0.0357 0 0.042 rpy=-0.87843 0 0; parent L4 -> L5

File: ros2_ur_ws/src/pallet_moveit_config/config/pallet.ros2_control.xacro (robot description, xacro)
@@ -8,4 +8,11 @@
                 <plugin>mock_components/GenericSystem</plugin>
             </hardware>
+            <joint name="j1">
+                <command_interface name="position"/>
+                <state_interface name="position">
+                  <param name="initial_value">${initial_positions['j1']}</param>
+                </state_interface>
+                <state_interface name="velocity"/>
+            </joint>
             <joint name="j2">
                 <command_interface name="position"/>
@@ -36,11 +43,4 @@
                 <state_interface name="velocity"/>
             </joint>
-            <joint name="j6">
-                <command_interface name="position"/>
-                <state_interface name="position">
-                  <param name="initial_value">${initial_positions['j6']}</param>
-                </state_interface>
-                <state_interface name="velocity"/>
-            </joint>
         </ros2_control>
     </xacro:macro>

Commit message: astra vision

File: ros2_ur_ws/src/pallet/urdf/pallet.urdf (robot description, URDF)
Before this commit: robot pallet, 9 links, 8 joints
Joints:
- joint j1: limit lower=-3.14 upper=3.14 effort=11 velocity=10.471976 -> lower=-3.14 upper=3.14 effort=5 velocity=10.471976
- joint j2: limit lower=-2.757620 upper=1.623156 effort=5 velocity=10.471976 -> lower=-2.757620 upper=1.623156 effort=11 velocity=10.471976
- joint j3: limit lower=-3.14 upper=0.802851 effort=1.8 velocity=10.471976 -> lower=-3.14 upper=0.802851 effort=5 velocity=10.471976

Commit message: Update MoveIt and RobStride control

File: ros2_ur_ws/src/pallet/urdf/pallet.urdf (robot description, URDF)
Before this commit: robot pallet, 11 links, 10 joints
Joints:
- joint J1: limit lower=-3.14 upper=3.14 effort=14 velocity=6.28 -> lower=-3.141592653589793 upper=3.141592653589793 effort=14 velocity=6.28; origin xyz=-0.0019451 0.043004 0 rpy=3.1416 -0.43861 -3.0964 -> xyz=-0.0019451 0.043004 0 rpy=-3.141585307179587 -0.4386100000000002 -3.0964
- joint J2: limit lower=-3.14 upper=3.14 effort=36 velocity=6.28 -> lower=-3.141592653589793 upper=3.141592653589793 effort=36 velocity=6.28; origin xyz=0.0133081654565508 0.11835224659499 -0.00768347290876137 rpy=2.6691912421104 0.23489083084202 -1.14340949773462 -> xyz=0.0133081654565508 0.11835224659499 -0.00768347290876137 rpy=-2.815387738468897 -0.4171744477814099 2.445921489969222
- joint J3: limit lower=-3.14 upper=3.14 effort=14 velocity=6.28 -> lower=-3.141592653589793 upper=3.141592653589793 effort=14 velocity=6.28; origin xyz=-0.213500000000005 0 0 rpy=2.98602758216798 -1.5707963267949 0 -> xyz=-0.213500000000005 0 0 rpy=-0.6266699393927205 -1.570796326794893 0
- joint J4: axis 0 0 1 -> 0 0 -1; limit lower=-3.14 upper=3.14 effort=5.5 velocity=6.28 -> lower=-3.141592653589793 upper=3.141592653589793 effort=5.5 velocity=6.28; origin xyz=-0.00799931400118803 -0.000150000000022965 0.167232496581933 rpy=0 0 0.616080039238196 -> xyz=-0.00799931400118803 -0.000150000000022965 0.167232496581933 rpy=0 0 0.05608003923819587
- joint J5: limit lower=-3.14 upper=3.14 effort=5.5 velocity=6.28 -> lower=-3.141592653589793 upper=3.141592653589793 effort=5.5 velocity=6.28; origin xyz=0 0 0.065768 rpy=-1.3579 0 3.1416 -> xyz=0 0 0.065768 rpy=-3.141488347732657 4.440892098500626e-16 -3.141585307179586
- joint J6: limit lower=-3.14 upper=3.14 effort=10 velocity=3.14 -> lower=-3.141592653589793 upper=3.141592653589793 effort=10 velocity=3.14; origin xyz=0.00205 0 -0.15365 rpy=-1.5708 0 -1.9447 -> xyz=0.00205 0 -0.15365 rpy=-1.570792653594452 -5.850140816221483e-09 1.198485307179575
- joint base_footprint_joint: origin xyz=0 0 0.0042247429751953 rpy=1.5707963267949 0 0 -> xyz=0.0001908929909025046 1.362578164557294e-10 3.325344132606295e-08 rpy=1.570796294509593 0.04519991100052101 -7.297706883235833e-10
- joint g_l: limit lower=-0.103 upper=0 effort=10 velocity=1.0 -> lower=0 upper=0.103 effort=10 velocity=1.0; origin xyz=0.007486 0.0031518 0.0082 rpy=0 0 -1.3963 -> xyz=0.007486 0.0031518 0.0082 rpy=0 0 -1.2933
- joint g_r: limit lower=0 upper=0.103 effort=10 velocity=1.0 -> lower=-0.103 upper=0 effort=10 velocity=1.0; origin xyz=-0.007486 0.0031518 0.0082 rpy=0 0 -1.7453 -> xyz=-0.007486 0.0031518 0.0082 rpy=0 0 -1.8483
