Commit message: refactor(pallet): align MoveIt with 6-axis J1-J6 and one-actuator gripper

File: ros2_ur_ws/src/pallet_moveit_config/config/pallet.ros2_control.xacro (robot description, xacro)
@@ -1,47 +1,23 @@
 <?xml version="1.0"?>
 <robot xmlns:xacro="http://www.ros.org/wiki/xacro">
-    <xacro:macro name="pallet_ros2_control" params="name initial_positions_file">
-        <xacro:property name="initial_positions" value="${load_yaml(initial_positions_file)['initial_positions']}"/>
-        <ros2_control name="${name}" type="system">
-            <hardware>
-                <!-- By default, set up controllers for simulation. This won't work on real hardware -->
-                <plugin>mock_components/GenericSystem</plugin>
-            </hardware>
-            <joint name="j1">
-                <command_interface name="position"/>
-                <state_interface name="position">
-                  <param name="initial_value">${initial_positions['j1']}</param>
-                </state_interface>
-                <state_interface name="velocity"/>
-            </joint>
-            <joint name="j2">
-                <command_interface name="position"/>
-                <state_interface name="position">
-                  <param name="initial_value">${initial_positions['j2']}</param>
-                </state_interface>
-                <state_interface name="velocity"/>
-            </joint>
-            <joint name="j3">
-                <command_interface name="position"/>
-                <state_interface name="position">
-                  <param name="initial_value">${initial_positions['j3']}</param>
-                </state_interface>
-                <state_interface name="velocity"/>
-            </joint>
-            <joint name="j4">
-                <command_interface name="position"/>
-                <state_interface name="position">
-                  <param name="initial_value">${initial_positions['j4']}</param>
-                </state_interface>
-                <state_interface name="velocity"/>
-            </joint>
-            <joint name="j5">
-                <command_interface name="position"/>
-                <state_interface name="position">
-                  <param name="initial_value">${initial_positions['j5']}</param>
-                </state_interface>
-                <state_interface name="velocity"/>
-            </joint>
-        </ros2_control>
-    </xacro:macro>
+  <xacro:macro name="pallet_ros2_control" params="name initial_positions_file">
+    <xacro:property name="initial_positions" value="${load_yaml(initial_positions_file)['initial_positions']}"/>
+    <ros2_control name="${name}" type="system">
+      <hardware><plugin>mock_components/GenericSystem</plugin></hardware>
+      <xacro:macro name="controlled_joint" params="joint_name">
+        <joint name="${joint_name}">
+          <command_interface name="position"/>
+          <state_interface name="position"><param name="initial_value">${initial_positions[joint_name]}</param></state_interface>
+          <state_interface name="velocity"/>
+        </joint>
+      </xacro:macro>
+      <xacro:controlled_joint joint_name="J1"/>
+      <xacro:controlled_joint joint_name="J2"/>
+      <xacro:controlled_joint joint_name="J3"/>
+      <xacro:controlled_joint joint_name="J4"/>
+      <xacro:controlled_joint joint_name="J5"/>
+      <xacro:controlled_joint joint_name="J6"/>
+      <xacro:controlled_joint joint_name="g_r"/>
+    </ros2_control>
+  </xacro:macro>
 </robot>

Commit message: restore(pallet): restore repository files to e8c099e5 pallet_change baseline

File: ros2_ur_ws/src/pallet_moveit_config/config/pallet.ros2_control.xacro (robot description, xacro)
@@ -1,23 +1,47 @@
 <?xml version="1.0"?>
 <robot xmlns:xacro="http://www.ros.org/wiki/xacro">
-  <xacro:macro name="pallet_ros2_control" params="name initial_positions_file">
-    <xacro:property name="initial_positions" value="${load_yaml(initial_positions_file)['initial_positions']}"/>
-    <ros2_control name="${name}" type="system">
-      <hardware><plugin>mock_components/GenericSystem</plugin></hardware>
-      <xacro:macro name="controlled_joint" params="joint_name">
-        <joint name="${joint_name}">
-          <command_interface name="position"/>
-          <state_interface name="position"><param name="initial_value">${initial_positions[joint_name]}</param></state_interface>
-          <state_interface name="velocity"/>
-        </joint>
-      </xacro:macro>
-      <xacro:controlled_joint joint_name="J1"/>
-      <xacro:controlled_joint joint_name="J2"/>
-      <xacro:controlled_joint joint_name="J3"/>
-      <xacro:controlled_joint joint_name="J4"/>
-      <xacro:controlled_joint joint_name="J5"/>
-      <xacro:controlled_joint joint_name="J6"/>
-      <xacro:controlled_joint joint_name="g_r"/>
-    </ros2_control>
-  </xacro:macro>
+    <xacro:macro name="pallet_ros2_control" params="name initial_positions_file">
+        <xacro:property name="initial_positions" value="${load_yaml(initial_positions_file)['initial_positions']}"/>
+        <ros2_control name="${name}" type="system">
+            <hardware>
+                <!-- By default, set up controllers for simulation. This won't work on real hardware -->
+                <plugin>mock_components/GenericSystem</plugin>
+            </hardware>
+            <joint name="j1">
+                <command_interface name="position"/>
+                <state_interface name="position">
+                  <param name="initial_value">${initial_positions['j1']}</param>
+                </state_interface>
+                <state_interface name="velocity"/>
+            </joint>
+            <joint name="j2">
+                <command_interface name="position"/>
+                <state_interface name="position">
+                  <param name="initial_value">${initial_positions['j2']}</param>
+                </state_interface>
+                <state_interface name="velocity"/>
+            </joint>
+            <joint name="j3">
+                <command_interface name="position"/>
+                <state_interface name="position">
+                  <param name="initial_value">${initial_positions['j3']}</param>
+                </state_interface>
+                <state_interface name="velocity"/>
+            </joint>
+            <joint name="j4">
+                <command_interface name="position"/>
+                <state_interface name="position">
+                  <param name="initial_value">${initial_positions['j4']}</param>
+                </state_interface>
+                <state_interface name="velocity"/>
+            </joint>
+            <joint name="j5">
+                <command_interface name="position"/>
+                <state_interface name="position">
+                  <param name="initial_value">${initial_positions['j5']}</param>
+                </state_interface>
+                <state_interface name="velocity"/>
+            </joint>
+        </ros2_control>
+    </xacro:macro>
 </robot>

File: ros2_ur_ws/src/pallet_moveit_config/config/pallet.urdf.xacro (robot description, xacro)
@@ -1,7 +1,10 @@
 <?xml version="1.0"?>
 <robot xmlns:xacro="http://www.ros.org/wiki/xacro" name="pallet">
-  <xacro:arg name="initial_positions_file" default="initial_positions.yaml"/>
-  <xacro:include filename="$(find pallet)/urdf/pallet_with_gripper.urdf"/>
-  <xacro:include filename="pallet.ros2_control.xacro"/>
-  <xacro:pallet_ros2_control name="FakeSystem" initial_positions_file="$(arg initial_positions_file)"/>
+    <xacro:arg name="initial_positions_file" default="initial_positions.yaml" />
+    <!-- Import pallet urdf file -->
+    <!-- Legacy five-axis controllers/SRDF are not compatible with the new CAD model. -->
+    <xacro:include filename="$(find pallet)/urdf/pallet_gripperless.urdf" />
+    <!-- Import control_xacro -->
+    <xacro:include filename="pallet.ros2_control.xacro" />
+    <xacro:pallet_ros2_control name="FakeSystem" initial_positions_file="$(arg initial_positions_file)"/>
 </robot>
